File: WaterSensor.kicad_pcb (KiCad board)
At the start: 2 copper layers, 304.8 x 304.8 mm, 8 parts, among them J2 Conn_01x03_Pin, Q1 2N3904

Commit message: Add pulldown resistor and update resistor values to bias a 3.3V output
Parts:
- added R3: 1.2k, Resistor_THT:R_Axial_DIN0204_L3.6mm_D1.6mm_P1.90mm_Vertical, B.Cu at (388.6, 71.1)
- J2: value Conn_01x03_Pin -> Main
- R1: value 100 -> 330
Routing:
- net PWR_SENSE: track 36101.0 -> 36098.9 mm, vias 0 -> 1

Commit message: Reverse changes as pulldown resistor is not needed
Parts:
- removed R3: 1.2k, Resistor_THT:R_Axial_DIN0204_L3.6mm_D1.6mm_P1.90mm_Vertical
- J2: value Main -> Conn_01x03_Pin
- R1: value 330 -> 100
Routing:
- net PWR_SENSE: track 36098.9 -> 36101.0 mm, vias 1 -> 0
