File: WaterSensor.kicad_pcb (KiCad board)
At the start: 2 copper layers, 304.8 x 304.8 mm, 8 parts, among them J2 Conn_01x03_Pin, Q1 2N3904

Commit message: Update resistor values based on calculations in README
Parts:
- J2: value Conn_01x03_Pin -> Main
- R1: value 100 -> 330k
- R2: value 100 -> 3.3k
Changed lines of the file:
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@@
 			)
 		)
-		(property "Footprint" ""
+		(property "Footprint" "MountingHole:MountingHole_2.5mm_Pad_Via"
 			(at 0 0 0)
 			(unlocked yes)
@@
 			)
 		)
-		(property "Description" "Mounting Hole with connection"
+		(property "Description" ""
 			(at 0 0 0)
 			(unlocked yes)
@@
 			)
 		)
+		(property ki_fp_filters "MountingHole*Pad*")
+		(sheetname "Root")
+		(sheetfile "WaterSensor.kicad_sch")
 		(attr exclude_from_pos_files)
 		(fp_circle
@@
 			)
 		)
-		(property "Footprint" ""
+		(property "Footprint" "MountingHole:MountingHole_2.5mm_Pad_Via"
 			(at 0 0 0)
 			(unlocked yes)
@@
 			)
 		)
-		(property "Description" "Mounting Hole with connection"
+		(property "Description" ""
 			(at 0 0 0)
 			(unlocked yes)
@@
 			)
 		)
+		(property ki_fp_filters "MountingHole*Pad*")
+		(sheetname "Root")
+		(sheetfile "WaterSensor.kicad_sch")
 		(attr exclude_from_pos_files)
 		(fp_circle
@@
 			)
 		)
-		(property "Footprint" ""
+		(property "Footprint" "MountingHole:MountingHole_2.5mm_Pad_Via"
 			(at 0 0 0)
 			(unlocked yes)
@@
 			)
 		)
-		(property "Description" "Mounting Hole with connection"
+		(property "Description" ""
 			(at 0 0 0)
 			(unlocked yes)
@@
 			)
 		)
+		(property ki_fp_filters "MountingHole*Pad*")
+		(sheetname "Root")
+		(sheetfile "WaterSensor.kicad_sch")
 		(attr exclude_from_pos_files)
 		(fp_circle
@@
 			)
 		)
-		(property "Footprint" ""
+		(property "Footprint" "MountingHole:MountingHole_2.5mm_Pad_Via"
 			(at 0 0 0)
 			(unlocked yes)
@@
 			)
 		)
-		(property "Description" "Mounting Hole with connection"
+		(property "Description" ""
 			(at 0 0 0)
 			(unlocked yes)
@@
 			)
 		)
+		(property ki_fp_filters "MountingHole*Pad*")
+		(sheetname "Root")
+		(sheetfile "WaterSensor.kicad_sch")
 		(attr exclude_from_pos_files)
 		(fp_circle
@@
 			)
 		)
-		(property "Value" "100"
+		(property "Value" "3.3k"
 			(at 0.95 -1.92 0)
 			(layer "B.Fab")
@@
 			)
 		)
-		(property "Footprint" ""
+		(property "Footprint" "Resistor_THT:R_Axial_DIN0204_L3.6mm_D1.6mm_P1.90mm_Vertical"
 			(at 0 0 180)
 			(unlocked yes)
@@
 			)
 		)
-		(property "Description" "Resistor"
+		(property "Description" ""
 			(at 0 0 180)
 			(unlocked yes)
@@
 			)
 		)
+		(property ki_fp_filters "R_*")
+		(sheetname "Root")
+		(sheetfile "WaterSensor.kicad_sch")
 		(attr through_hole)
 		(fp_arc
@@
 			)
 		)
-		(property "Value" "Conn_01x03_Pin"
+		(property "Value" "Main"
 			(at 0 -7.41 90)
 			(layer "B.Fab")
@@
 			)
 		)
-		(property "Footprint" ""
+		(property "Footprint" "Connector_PinHeader_2.54mm:PinHeader_1x03_P2.54mm_Vertical"
 			(at 0 0 -90)
 			(unlocked yes)
@@
 			)
 		)
-		(property "Description" "Generic connector, single row, 01x03, script generated"
+		(property "Description" ""
 			(at 0 0 -90)
 			(unlocked yes)
@@
 			)
 		)
+		(property ki_fp_filters "Connector*:*_1x??_*")
+		(sheetname "Root")
+		(sheetfile "WaterSensor.kicad_sch")
 		(attr through_hole)
 		(fp_line
@@
 			)
 		)
-		(property "Value" "100"
+		(property "Value" "330k"
 			(at 0.95 -1.92 90)
 			(layer "B.Fab")
@@
 			)
 		)
-		(property "Footprint" ""
+		(property "Footprint" "Resistor_THT:R_Axial_DIN0204_L3.6mm_D1.6mm_P1.90mm_Vertical"
 			(at 0 0 -90)
 			(unlocked yes)
@@
 			)
 		)
-		(property "Description" "Resistor"
+		(property "Description" ""
 			(at 0 0 -90)
 			(unlocked yes)
@@
 			)
 		)
+		(property ki_fp_filters "R_*")
+		(sheetname "Root")
+		(sheetfile "WaterSensor.kicad_sch")
 		(attr through_hole)
 		(fp_arc
@@
 			)
 		)
-		(property "Footprint" ""
+		(property "Footprint" "Package_TO_SOT_THT:TO-92_Inline"
 			(at 0 0 -90)
 			(unlocked yes)
@@
 			)
 		)
-		(property "Datasheet" ""
+		(property "Datasheet" "https://www.onsemi.com/pub/Collateral/2N3903-D.PDF"
 			(at 0 0 -90)
 			(unlocked yes)
@@
 			)
 		)
-		(property "Description" "0.2A Ic, 40V Vce, Small Signal NPN Transistor, TO-92"
+		(property "Description" ""
 			(at 0 0 -90)
 			(unlocked yes)
@@
 			)
 		)
+		(property ki_fp_filters "TO?92*")
+		(sheetname "Root")
+		(sheetfile "WaterSensor.kicad_sch")
 		(attr through_hole)
 		(fp_line
@@
 		(polygon
 			(pts
-				(xy 436.88 41.91) (xy 123.19 40.64) (xy 121.92 355.6) (xy 439.42 355.6)
+				(xy 124.46 355.6) (xy 436.88 354.33) (xy 434.34 41.91) (xy 393.7 41.91) (xy 393.7 53.34) (xy 403.86 53.34)
+				(xy 403.86 58.42) (xy 401.32 63.5) (xy 396.24 71.12) (xy 391.16 71.12) (xy 391.16 68.58) (xy 384.81 68.58)
+				(xy 384.81 60.96) (xy 392.43 60.96) (xy 392.43 53.34) (xy 393.7 53.34) (xy 393.7 41.91) (xy 123.19 41.91)
 			)
 		)
